File: nora-b106-board.kicad_sch (KiCad schematic)
At the start: 15 parts, among them J1 TYPE-C-31-M-12, J2 SWD / PICO, J3 GPIO 3V3, SW1 RESET, U1 NORA-B106-00B, U2 XC6206P332MR-G, U3 USBLC6-2SC6

Commit message: Expose six more GPIOs on optional headers in revision C
Parts:
- added J4: EXTRA GPIO, Breakout:PinHeader_1x04_P2.54mm_Vertical, symbol Connector_Generic:Conn_01x04
- added J5: EXTRA GPIO, Breakout:PinHeader_1x02_P2.54mm_Vertical, symbol Connector_Generic:Conn_01x02
Connections:
- net P0.15: now reaches U1.D1 (P0.15)
- net P0.15: now also J5.2 (Pin_2)
- net P0.18: now reaches U1.E1 (P0.18)
- net P0.18: now also J5.1 (Pin_1)
- net P1.05: now reaches U1.E9 (P1.05)
- net P1.05: now also J4.4 (Pin_4)
- net P1.15: now reaches U1.F9 (P1.15)
- net P1.15: now also J4.3 (Pin_3)
- net P1.11: now reaches U1.H9 (P1.11)
- net P1.11: now also J4.2 (Pin_2)
- net P0.31: now reaches U1.J9 (P0.31)
- net P0.31: now also J4.1 (Pin_1)
- no-connect marks 49 -> 43
Other:
- note added: "J2: 3V3 sense, GND, CLK, DIO, RESET. Pico GP2 -> CLK; GP3 -> DIO; GP1 -> RESET. Do not connect Pico 3V3 when USB-powered. J4: P0.31 / P1.11 / P1.15 / P1.05. GPIO only."
- note added: "J3/J4/J5: 3V3 logic only; no 5V-tolerant GPIO. Use the internal LF RC clock; no 32k crystal. All unbroken-out GPIO and reserved pads NC."
- note removed: "J2: 3V3 sense, GND, CLK, DIO, RESET. Pico GP2 -> CLK; GP3 -> DIO; GP1 -> RESET. Do not connect Pico 3V3 when USB-powered."
- note removed: "J3: 3V3 logic only; no 5V-tolerant GPIO. Use the internal LF RC clock; no 32k crystal. All unbroken-out GPIO and reserved pads NC."

Commit message: Consolidate GPIOs into one right-edge header in revision D
Parts:
- removed J4: EXTRA GPIO, Breakout:PinHeader_1x04_P2.54mm_Vertical, symbol Connector_Generic:Conn_01x04
- removed J5: EXTRA GPIO, Breakout:PinHeader_1x02_P2.54mm_Vertical, symbol Connector_Generic:Conn_01x02
- J3: value GPIO 3V3 -> GPIO / 3V3; footprint Breakout:PinHeader_1x08_P2.54mm_Vertical -> Breakout:PinHeader_1x14_P2.54mm_Vertical; symbol Connector_Generic:Conn_01x08 -> Connector_Generic:Conn_01x14
Connections:
- net P0.04_AIN0: now also J3.11 (Pin_11); no longer J3.5 (Pin_5)
- net P0.05_AIN1: now also J3.12 (Pin_12); no longer J3.6 (Pin_6)
- net P0.15: now also J3.4 (Pin_4)
- net P0.18: now also J3.3 (Pin_3)
- net P0.31: now also J3.5 (Pin_5)
- net P1.02_SDA: now also J3.13 (Pin_13); no longer J3.7 (Pin_7)
- net P1.03_SCL: now also J3.14 (Pin_14); no longer J3.8 (Pin_8)
- net P1.05: now also J3.8 (Pin_8)
- net P1.11: now also J3.6 (Pin_6)
- net P1.12_TX: now also J3.9 (Pin_9); no longer J3.3 (Pin_3)
- net P1.13_RX: now also J3.10 (Pin_10); no longer J3.4 (Pin_4)
- net P1.15: now also J3.7 (Pin_7)
Other:
- note added: "J2: 3V3 sense, GND, CLK, DIO, RESET. Pico GP2 -> CLK; GP3 -> DIO; GP1 -> RESET. Do not connect Pico 3V3 when USB-powered. J3: single 1x14 GPIO/power header; see pin labels."
- note added: "J3: 3V3 logic only; no 5V-tolerant GPIO. Use the internal LF RC clock; no 32k crystal. All unbroken-out GPIO and reserved pads NC."
- note removed: "J2: 3V3 sense, GND, CLK, DIO, RESET. Pico GP2 -> CLK; GP3 -> DIO; GP1 -> RESET. Do not connect Pico 3V3 when USB-powered. J4: P0.31 / P1.11 / P1.15 / P1.05. GPIO only."
- note removed: "J3/J4/J5: 3V3 logic only; no 5V-tolerant GPIO. Use the internal LF RC clock; no 32k crystal. All unbroken-out GPIO and reserved pads NC."
